Commit message: Started testing the new_model, so far so good. There's also a lot of errors in the urdf file and the spawn position fo the ball, still need to doublecheck that.

File: Reinforcement Learning/URDF/new_pong2.urdf (robot description, URDF)
Before this commit: robot robot_test, 11 links, 10 joints
Links:
- link player_sensor: geometry collision box size=0.3 0.4 0.02; visual box size=0.3 0.4 0.02
- link playerwall_link: geometry collision box size=0.3 0.01 0.3; visual box size=0.3 0.01 0.3
- link robot_sensor: geometry collision box size=0.3 0.4 0.02; visual box size=0.3 0.4 0.02
- link robotwall_link: geometry collision box size=0.3 0.01 0.3; visual box size=0.3 0.01 0.3
- link striker2_body: geometry collision box size=0.1 0.10 0.08; visual box size=0.1 0.10 0.08
- link striker2_link: geometry collision cylinder length=0.0801 radius=0.06; visual cylinder length=0.0801 radius=0.06
- link striker_link: geometry collision cylinder length=0.0801 radius=0.06; visual cylinder length=0.0801 radius=0.06
Joints:
- joint prismatic2_joint: limit lower=-0.1 upper=0.1 -> lower=-0.09 upper=0.09
- joint prismatic_joint: limit lower=-0.1 upper=0.1 effort=100 velocity=1.0 -> lower=-0.09 upper=0.09 effort=100 velocity=1.0
- joint striker2_joint: limit lower=0 upper=0.015 -> lower=-0.015 upper=0
