Commit message: Changed shoot penalty from -0.01 to -0.0001.

File: Reinforcement_Learning/URDF/pong2.urdf (robot description, URDF)
Before this commit: robot robot_test, 9 links, 8 joints
Links:
- link base_link: mass 24.072 -> 24.072000000000003
- link leftwall_link: mass 4.956 -> 4.9559999999999995
- link rightwall_link: mass 4.956 -> 4.9559999999999995
